File: Domowy Sterownik GSM.sch (KiCad schematic (older format))
At the start: 97 parts

Commit message: 18-03-2015
Parts:
- removed D? (x4): SS24, ~, symbol DIODE
- added D? (x4): SS24, ~, symbol DIODESCH
- added IC?: TLP281-4, SOP16, symbol TLP291-4
- added P?: WE1, symbol CONN_2
- added P?: WE2, symbol CONN_2
- added P?: WE3, symbol CONN_2
- added P?: WE4, symbol CONN_2
- added Q? (x2): BC817, ~, symbol NPN
- added R? (x3): 470R, ~, symbol R
- added R? (x6): 4,7k, ~, symbol R
- added RV?: POT, ~, symbol POT
- added S?: LCD, ~, symbol LCD
- added SP?: TMB12A05, ~, symbol SPEAKER
- added SW?: OK, ~, symbol SW_PUSH_SMALL
- added SW?: UP, ~, symbol SW_PUSH_SMALL
- added SW?: DN, ~, symbol SW_PUSH_SMALL
- added SW?: LT, ~, symbol SW_PUSH_SMALL
- added SW?: RT, ~, symbol SW_PUSH_SMALL
- R? (x4): value R -> 4,7k
- R?: value R -> 470R
Connections:
- net labels added: +9V, BUZZ, D4, D5, D6, D7, DN, E, LCD_BL, LT, OK, R/W, RS, RT, UP, WE1, WE2, WE3, WE4
- wire segments 234 -> 301
- no-connect marks 0 -> 4
Other:
- moved on the sheet: IC?, IC?A, R?

Commit message: 21-03-2015
Parts:
- added D?: PWR, ~, symbol LED
- added D?: ERR, ~, symbol LED
- added D?: TR1, ~, symbol LED
- added D?: TR2, ~, symbol LED
- added D?: TR3, ~, symbol LED
- added D?: TR4, ~, symbol LED
- added D?: RE1, ~, symbol LED
- added D?: RE2, ~, symbol LED
- added D?: RE3, ~, symbol LED
- added D?: RE4, ~, symbol LED
- added P?: 1_wire, symbol CONN_2
- added Q?: IRLML2502, ~, symbol MOSFET_N
- added R?: 560R, ~, symbol R
- added R?: 47R/1W, ~, symbol R
- added R?: 1k, ~, symbol R
- added R?: 5k, ~, symbol R
- added R? (x10): 2,2k, ~, symbol R
- added R?: 4,7k, ~, symbol R
- added RV?: 10k, ~, symbol POT
- added U?: MQ-2, symbol MQ-2
- added U?: MD-PIR, symbol MD-PIR
- added U?: DHT-11, ~, symbol DHT-11
- VR?: value VR -> V07N361-F
Connections:
- net labels added: DQ, ERR, GAS, HUM, PIR, PULL_UP
- wire segments 301 -> 355
- no-connect marks 4 -> 5
Other:
- moved on the sheet: C?, IC?, L?, Q?, R?, RV?, S?, SP?, SW?, X?

Commit message: 24-03-2015
Parts:
- removed R? (x2): R, ~, symbol R
- removed U?: TL081, symbol TL081
- added P12: MODUL, symbol CONN_10
- C13: renamed from C?; value 100nF/400V -> 100n/400V
- gave numbers to parts that had none: 145
Connections:
- net labels added: ZERO
- wire segments 355 -> 346
Other:
- moved on the sheet: IC6, R13, R14, R27

Commit message: Revert "Revert "28-03-2015""
This reverts commit a35226c248e7f072a54264f71b0718be7540caac.
Parts:
- removed IC3, IC4: LTV817, DIP4, symbol PC817
- removed IC6: TLP180, SOP4, symbol TLP290
- removed R27: 10k, ~, symbol R
- removed R46, R47, R48, R49, R50: 4,7k, ~, symbol R
- removed SW2: OK, ~, symbol SW_PUSH_SMALL
- removed SW3: UP, ~, symbol SW_PUSH_SMALL
- removed SW4: DN, ~, symbol SW_PUSH_SMALL
- removed SW5: LT, ~, symbol SW_PUSH_SMALL
- removed SW6: RT, ~, symbol SW_PUSH_SMALL
- removed U1: BRIDGE_SMALL, symbol BRIDGE_SMALL
- removed U11: MD-PIR, symbol MD-PIR
- added C14: 470u, symbol CP1
- added C15, C16, C17, C18, C20: 100n, ~, symbol C
- added C19: 22u/T, ~, symbol CP1
- added CON1: PROG, AVR-ISP-10, symbol AVR-ISP-10
- added CON2: DEBUG, AVR-JTAG-10, symbol AVR-JTAG-10
- added D15, D16, D17, D18: S3M, ~, symbol DIODE
- added IC3, IC4: TLP180, MFSOP6, symbol TLP185
- added P13: KEYS, symbol CONN_8
- added R11: 33k/2W, ~, symbol R
- added R23: 10k, ~, symbol R
- added RV3: 10k, ~, symbol POT
- added U1: 74HC595, ~, symbol 74LS595
- C1: value 220u -> 470u
- C4: value 22u -> 100u
- F1: value FUSE -> 8A
- F2: value FUSE -> 100mA
- R12: value 68k/2W -> 33k/2W
- RV1: value POT -> 10k
- T1: value TRANSFO -> 230V/9V
- X1: value CRYSTAL -> 16MHz
Connections:
- net R/W is gone; now on net DGND: S1.5 (R/W)
- net WE1 is gone; now on net IN1: IC8.16, R31.2
- net WE2 is gone; now on net IN2: IC8.14, R32.2
- net WE3 is gone; now on net IN3: IC8.12, R33.2
- net WE4 is gone; now on net IN4: IC8.10, R34.2
- net +5V: now also P12.1 (P1), C15.1, C16.1, C17.1, C18.1, C19.1, C20.1, CON1.2, CON2.4, P13.1 (P1), U1.10 (SRCLR), U1.16 (VCC)
- net +9V: now also C14.1, D15.2 (K), D16.2 (K)
- net BUZZ: now also IC9.16 ((OC2)PD7)
- net D4: now also IC9.34 ((ADC3)PA3)
- net D5: now also IC9.33 ((ADC4)PA4)
- net D6: now also IC9.32 ((ADC5)PA5)
- net D7: now also IC9.31 ((ADC6)PA6)
- net DGND: now also P12.2 (P2), C14.2, C15.2, C16.2, C17.2, C18.2, C19.2, C20.2, CON1.10, CON1.3, CON1.4, CON1.6, CON1.8, CON2.10, CON2.2, D17.1 (A), D18.1 (A), IC3.4, IC4.4, P13.7 (P7), P13.8 (P8), RV3.1, U1.13 (G), U1.8 (GND)
- net DN: now also IC9.13 ((OC1B)PD4), P13.4 (P4)
- net DQ: now also IC9.41 ((T1)PB1), R54.2
- net E: now also IC9.35 ((ADC2)PA2)
- net ERR: now also IC9.19 ((SCL)PC0)
- net GAS: now also IC9.37 ((ADC0)PA0)
- net HUM: now also IC9.26 ((TOSC2)PC7)
- net L: now also R11.2; no longer R12.1
- net LCD_BL: now also IC9.30 ((ADC7)PA7)
- net LT: now also IC9.14 ((OC1A)PD5), P13.5 (P5)
- net N: now also IC3.3, IC4.1
- net OK: now also IC9.11 ((INT0)PD2), P13.2 (P2)
- net PULL_UP: now also IC9.40 ((T0/XCK)PB0)
- net RE1: now also U1.4 (QE)
- net RE2: now also U1.5 (QF)
- net RE3: now also U1.6 (QG)
- net RE4: now also U1.7 (QH)
- net RS: now also IC9.36 ((ADC1)PA1)
- net RT: now also IC9.15 ((ICP)PD6), P13.6 (P6)
- net TR1: now also U1.15 (QA)
- net TR2: now also U1.1 (QB)
- net TR3: now also U1.2 (QC)
- net TR4: now also U1.3 (QD)
- net TR5: now also IC9.25 ((TOSC1)PC6)
- net UP: now also IC9.12 ((INT1)PD3), P13.3 (P3)
- net ZERO: now also IC3.6, IC4.6
- net MOSI: now reaches IC9.1 ((MOSI)PB5)
- net MOSI: now also P12.6 (P6), CON1.1, U1.14 (SER)
- net TX: now reaches IC9.10 ((TXD)PD1)
- net TX: now also P12.4 (P4)
- net MISO: now reaches IC9.2 ((MISO)PB6)
- net MISO: now also P12.7 (P7), CON1.9
- net WR: now reaches IC9.20 ((SDA)PC1)
- net WR: now also U1.12 (RCLK)
- net IN1: now reaches IC9.21 ((TCK)PC2)
- net IN1: now also CON2.1
- net IN2: now reaches IC9.22 ((TMS)PC3)
- net IN2: now also CON2.5
- net IN3: now reaches IC9.23 ((TDO)PC4)
- net IN3: now also CON2.3
- net IN4: now reaches IC9.24 ((TDI)PC5)
- net IN4: now also CON2.9
- net SCK: now reaches IC9.3 ((SCK)PB7)
- net SCK: now also P12.8 (P8), CON1.7, U1.11 (SRCLK)
- net RST: now reaches IC9.4 (~RESET), R29.2, SW1.2
- net RST: now also P12.3 (P3), CON1.5, CON2.6
- net at IC9.42 ((AIN0/INT2)PB2), R14.2: now also R23.1
- net ~SS: now reaches IC9.44 ((~SS~)PB4)
- net ~SS: now also P12.9 (P9)
- net RX: now reaches IC9.9 ((RXD)PD0)
- net RX: now also P12.5 (P5)
- net at T1.3 (SA): now also D16.1 (A), D18.2 (K)
- net at T1.4 (SB): now also D15.1 (A), D17.2 (K)
- net at R12.2: now also IC3.1, IC4.3
- new net: R11.1, R12.1
- new net: R23.2, RV3.2, RV3.3
- no-connect marks 5 -> 9
Other:
- moved on the sheet: C1, C10, C12, C2, C3, C4, C7, C9, D1, D2, F2, IC9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

Commit message: Revert "28-03-2015"
This reverts commit 6328e8af113ad8d7fc7daed5852ae822de97dd85.
Parts:
- removed C14: 470u, symbol CP1
- removed C15, C16, C17, C18, C20: 100n, ~, symbol C
- removed C19: 22u/T, ~, symbol CP1
- removed CON1: PROG, AVR-ISP-10, symbol AVR-ISP-10
- removed CON2: DEBUG, AVR-JTAG-10, symbol AVR-JTAG-10
- removed D15, D16, D17, D18: S3M, ~, symbol DIODE
- removed IC3, IC4: TLP180, MFSOP6, symbol TLP185
- removed P13: KEYS, symbol CONN_8
- removed R11: 33k/2W, ~, symbol R
- removed R23: 10k, ~, symbol R
- removed RV3: 10k, ~, symbol POT
- removed U1: 74HC595, ~, symbol 74LS595
- added IC3, IC4: LTV817, DIP4, symbol PC817
- added IC6: TLP180, SOP4, symbol TLP290
- added R27: 10k, ~, symbol R
- added R46, R47, R48, R49, R50: 4,7k, ~, symbol R
- added SW2: OK, ~, symbol SW_PUSH_SMALL
- added SW3: UP, ~, symbol SW_PUSH_SMALL
- added SW4: DN, ~, symbol SW_PUSH_SMALL
- added SW5: LT, ~, symbol SW_PUSH_SMALL
- added SW6: RT, ~, symbol SW_PUSH_SMALL
- added U1: BRIDGE_SMALL, symbol BRIDGE_SMALL
- added U11: MD-PIR, symbol MD-PIR
- C1: value 470u -> 220u
- C4: value 100u -> 22u
- F1: value 8A -> FUSE
- F2: value 100mA -> FUSE
- R12: value 33k/2W -> 68k/2W
- RV1: value 10k -> POT
- T1: value 230V/9V -> TRANSFO
- X1: value 16MHz -> CRYSTAL
Connections:
- net +5V: now also R46.1, R47.1, R48.1, R49.1, R50.1, U11.3 (VDD); no longer P12.1 (P1)
- net +9V: now also U1.4
- net BUZZ: no longer IC9.16 ((OC2)PD7)
- net D4: no longer IC9.34 ((ADC3)PA3)
- net D5: no longer IC9.33 ((ADC4)PA4)
- net D6: no longer IC9.32 ((ADC5)PA5)
- net D7: no longer IC9.31 ((ADC6)PA6)
- net DGND: now also IC3.3, IC4.3, R27.2, SW2.2, SW3.2, SW4.2, SW5.2, SW6.2, U1.3, U11.1 (GND); no longer P12.2 (P2), S1.5 (R/W)
- net DN: now also R48.2, SW4.1; no longer IC9.13 ((OC1B)PD4)
- net DQ: no longer IC9.41 ((T1)PB1), R54.2
- net E: no longer IC9.35 ((ADC2)PA2)
- net ERR: no longer IC9.19 ((SCL)PC0)
- net GAS: no longer IC9.37 ((ADC0)PA0)
- net HUM: no longer IC9.26 ((TOSC2)PC7)
- net L: now also R12.1
- net LCD_BL: no longer IC9.30 ((ADC7)PA7)
- net LT: now also R49.2, SW5.1; no longer IC9.14 ((OC1A)PD5)
- net N: now also IC3.2, IC4.1
- net OK: now also R46.2, SW2.1; no longer IC9.11 ((INT0)PD2)
- net PULL_UP: no longer IC9.40 ((T0/XCK)PB0)
- net RS: no longer IC9.36 ((ADC1)PA1)
- net RT: now also R50.2, SW6.1; no longer IC9.15 ((ICP)PD6)
- net TR5: no longer IC9.25 ((TOSC1)PC6)
- net UP: now also R47.2, SW3.1; no longer IC9.12 ((INT1)PD3)
- net ZERO: now also IC3.4, IC4.4
- net at IC9.42 ((AIN0/INT2)PB2), R14.2: now also R27.1
- net at T1.3 (SA): now also U1.2
- net at T1.4 (SB): now also U1.1
- net at R12.2: now also IC3.1, IC4.2
- net IN1 renamed WE1
- net WE1: no longer IC9.21 ((TCK)PC2)
- net IN2 renamed WE2
- net WE2: no longer IC9.22 ((TMS)PC3)
- net IN3 renamed WE3
- net WE3: no longer IC9.23 ((TDO)PC4)
- net IN4 renamed WE4
- net WE4: no longer IC9.24 ((TDI)PC5)
- net MISO: no longer names the net of IC9.2 ((MISO)PB6)
- net MISO: no longer P12.7 (P7)
- net MOSI: no longer names the net of IC9.1 ((MOSI)PB5)
- net MOSI: no longer P12.6 (P6)
- net RST: no longer names the net of IC9.4 (~RESET), R29.2, SW1.2
- net RST: no longer P12.3 (P3)
- net RX: no longer names the net of IC9.9 ((RXD)PD0)
- net RX: no longer P12.5 (P5)
- net SCK: no longer names the net of IC9.3 ((SCK)PB7)
- net SCK: no longer P12.8 (P8)
- net TX: no longer names the net of IC9.10 ((TXD)PD1)
- net TX: no longer P12.4 (P4)
- net WR: no longer names the net of IC9.20 ((SDA)PC1)
- net ~SS: no longer names the net of IC9.44 ((~SS~)PB4)
- net ~SS: no longer P12.9 (P9)
- new net PIR: U11.2 (OUT)
- new net R/W: S1.5 (R/W)
- no-connect marks 9 -> 5
Other:
- moved on the sheet: C1, C10, C12, C2, C3, C4, C7, C9, D1, D2, F2, IC9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
